File: breakout-qfn/caravel-breakout-qfn.kicad_pcb (KiCad board)
At the start: 2 copper layers, 45 x 57.5 mm, 83 parts, among them CON1 REF-182665-01, CON2 REF-182665-01, CON3 73251-1352, U1 Caravel_QFN_TT4

Commit message: TT123 "legacy" breakout rework
Parts:
- removed the REF** at (90.5, 54.8)
- removed the REF** at (72.8, 32.5)
- removed the REF** at (65.0, 19.6)
- removed the REF** at (63.0, 37.0)
- removed the REF** at (63.0, 33.0)
- removed the REF** at (50.5, 68.2)
- removed the REF** at (85.4, 61.1)
- removed the REF** at (64.8, 56.1)
- removed the REF** at (63.0, 26.0)
- removed the REF** at (67.7, 55.0)
- removed the REF** at (89.3, 38.6)
- removed the REF** at (90.5, 23.6)
- removed the REF** at (87.3, 51.4)
- removed the REF** at (90.5, 28.2)
- removed the REF** at (64.8, 59.4)
- removed the REF** at (48.7, 36.5)
- removed the REF** at (63.0, 23.0)
- removed the REF** at (55.6, 36.1)
- removed the REF** at (77.4, 20.6)
- removed the REF** at (78.0, 53.0)
- removed the REF** at (72.8, 29.1)
- removed the REF** at (80.4, 64.2)
- removed the REF** at (71.7, 61.0)
- removed the REF** at (78.0, 57.5)
- removed the REF** at (66.0, 35.9)
- removed the REF** at (62.9, 41.2)
- removed the REF** at (78.0, 68.5)
- removed the REF** at (68.0, 30.8)
- removed the REF** at (63.0, 29.5)
- removed the REF** at (80.8, 51.4)
- removed the REF** at (70.0, 35.5)
- removed the REF** at (79.7, 29.1)
- removed the REF** at (78.0, 61.0)
- removed the REF** at (58.6, 41.2)
- removed the REF** at (72.5, 56.6)
- removed the REF** at (72.8, 24.4)
- removed the REF** at (91.2, 63.8)
- removed the REF** at (70.8, 55.0)
- added STITCH: StitchingVia-0.3mm, flyingcarsfootprints:StitchingVia-0.3mm, F.Cu at (74.2, 18.2)
- added STITCH: StitchingVia-0.3mm, flyingcarsfootprints:StitchingVia-0.3mm, F.Cu at (48.8, 50.1)
- added STITCH: StitchingVia-0.3mm, flyingcarsfootprints:StitchingVia-0.3mm, F.Cu at (74.9, 24.3)
- added STITCH: StitchingVia-0.3mm, flyingcarsfootprints:StitchingVia-0.3mm, F.Cu at (73.8, 61.1)
- added STITCH: StitchingVia-0.3mm, flyingcarsfootprints:StitchingVia-0.3mm, F.Cu at (74.9, 26.4)
- added STITCH: StitchingVia-0.3mm, flyingcarsfootprints:StitchingVia-0.3mm, F.Cu at (49.0, 25.5)
- added STITCH: StitchingVia-0.3mm, flyingcarsfootprints:StitchingVia-0.3mm, F.Cu at (74.9, 30.5)
- added STITCH: StitchingVia-0.3mm, flyingcarsfootprints:StitchingVia-0.3mm, F.Cu at (53.9, 33.6)
- added STITCH: StitchingVia-0.3mm, flyingcarsfootprints:StitchingVia-0.3mm, F.Cu at (51.5, 53.9)
- added STITCH: StitchingVia-0.3mm, flyingcarsfootprints:StitchingVia-0.3mm, F.Cu at (51.5, 56.5)
- added STITCH: StitchingVia-0.3mm, flyingcarsfootprints:StitchingVia-0.3mm, F.Cu at (72.2, 51.6)
- added STITCH: StitchingVia-0.3mm, flyingcarsfootprints:StitchingVia-0.3mm, F.Cu at (49.0, 21.0)
- added STITCH: StitchingVia-0.3mm, flyingcarsfootprints:StitchingVia-0.3mm, F.Cu at (70.0, 30.5)
- added STITCH: StitchingVia-0.3mm, flyingcarsfootprints:StitchingVia-0.3mm, F.Cu at (51.5, 61.5)
- added STITCH: StitchingVia-0.3mm, flyingcarsfootprints:StitchingVia-0.3mm, F.Cu at (81.0, 18.2)
- added STITCH: StitchingVia-0.3mm, flyingcarsfootprints:StitchingVia-0.3mm, F.Cu at (79.7, 59.0)
- added STITCH: StitchingVia-0.3mm, flyingcarsfootprints:StitchingVia-0.3mm, F.Cu at (59.8, 18.2)
- added STITCH: StitchingVia-0.3mm, flyingcarsfootprints:StitchingVia-0.3mm, F.Cu at (65.3, 24.3)
- added STITCH: StitchingVia-0.3mm, flyingcarsfootprints:StitchingVia-0.3mm, F.Cu at (51.5, 51.2)
- added STITCH: StitchingVia-0.3mm, flyingcarsfootprints:StitchingVia-0.3mm, F.Cu at (90.0, 18.2)
- added STITCH: StitchingVia-0.3mm, flyingcarsfootprints:StitchingVia-0.3mm, F.Cu at (73.8, 59.0)
- added STITCH: StitchingVia-0.3mm, flyingcarsfootprints:StitchingVia-0.3mm, F.Cu at (92.2, 21.0)
- added STITCH: StitchingVia-0.3mm, flyingcarsfootprints:StitchingVia-0.3mm, F.Cu at (62.7, 23.0)
- added STITCH: StitchingVia-0.3mm, flyingcarsfootprints:StitchingVia-0.3mm, F.Cu at (66.8, 18.2)
- added STITCH: StitchingVia-0.3mm, flyingcarsfootprints:StitchingVia-0.3mm, F.Cu at (65.3, 27.9)
- added STITCH: StitchingVia-0.3mm, flyingcarsfootprints:StitchingVia-0.3mm, F.Cu at (80.6, 27.9)
- added STITCH: StitchingVia-0.3mm, flyingcarsfootprints:StitchingVia-0.3mm, F.Cu at (71.9, 24.3)
- added STITCH: StitchingVia-0.3mm, flyingcarsfootprints:StitchingVia-0.3mm, F.Cu at (51.2, 18.2)
- added STITCH1: StitchingVia-0.3mm, flyingcarsfootprints:StitchingVia-0.3mm, F.Cu at (92.2, 23.5)
- added STITCH10: StitchingVia-0.3mm, flyingcarsfootprints:StitchingVia-0.3mm, F.Cu at (49.1, 68.9)
- added STITCH10: StitchingVia-0.3mm, flyingcarsfootprints:StitchingVia-0.3mm, F.Cu at (77.0, 64.5)
- added STITCH10: StitchingVia-0.3mm, flyingcarsfootprints:StitchingVia-0.3mm, F.Cu at (52.5, 69.3)
- added STITCH10: StitchingVia-0.3mm, flyingcarsfootprints:StitchingVia-0.3mm, F.Cu at (91.8, 69.0)
- added STITCH11: StitchingVia-0.3mm, flyingcarsfootprints:StitchingVia-0.3mm, F.Cu at (55.0, 69.3)
- added STITCH12: StitchingVia-0.3mm, flyingcarsfootprints:StitchingVia-0.3mm, F.Cu at (57.6, 69.3)
- added STITCH13: StitchingVia-0.3mm, flyingcarsfootprints:StitchingVia-0.3mm, F.Cu at (60.1, 69.3)
- added STITCH14: StitchingVia-0.3mm, flyingcarsfootprints:StitchingVia-0.3mm, F.Cu at (62.7, 69.3)
- added STITCH15: StitchingVia-0.3mm, flyingcarsfootprints:StitchingVia-0.3mm, F.Cu at (65.2, 69.3)
- added STITCH16: StitchingVia-0.3mm, flyingcarsfootprints:StitchingVia-0.3mm, F.Cu at (48.8, 54.1)
- added STITCH17: StitchingVia-0.3mm, flyingcarsfootprints:StitchingVia-0.3mm, F.Cu at (70.3, 69.3)
- added STITCH18: StitchingVia-0.3mm, flyingcarsfootprints:StitchingVia-0.3mm, F.Cu at (48.8, 58.1)
- added STITCH19: StitchingVia-0.3mm, flyingcarsfootprints:StitchingVia-0.3mm, F.Cu at (75.4, 69.3)
- added STITCH2: StitchingVia-0.3mm, flyingcarsfootprints:StitchingVia-0.3mm, F.Cu at (92.2, 26.1)
- added STITCH20: StitchingVia-0.3mm, flyingcarsfootprints:StitchingVia-0.3mm, F.Cu at (77.9, 69.3)
- added STITCH21: StitchingVia-0.3mm, flyingcarsfootprints:StitchingVia-0.3mm, F.Cu at (80.4, 69.3)
- added STITCH22: StitchingVia-0.3mm, flyingcarsfootprints:StitchingVia-0.3mm, F.Cu at (83.0, 69.3)
- added STITCH23: StitchingVia-0.3mm, flyingcarsfootprints:StitchingVia-0.3mm, F.Cu at (85.5, 69.3)
- added STITCH24: StitchingVia-0.3mm, flyingcarsfootprints:StitchingVia-0.3mm, F.Cu at (88.1, 69.3)
- added STITCH25: StitchingVia-0.3mm, flyingcarsfootprints:StitchingVia-0.3mm, F.Cu at (48.8, 62.1)
- added STITCH26: StitchingVia-0.3mm, flyingcarsfootprints:StitchingVia-0.3mm, F.Cu at (48.8, 66.1)
- added STITCH27: StitchingVia-0.3mm, flyingcarsfootprints:StitchingVia-0.3mm, F.Cu at (70.8, 61.1)
- added STITCH27: StitchingVia-0.3mm, flyingcarsfootprints:StitchingVia-0.3mm, F.Cu at (70.8, 59.0)
- added STITCH28: StitchingVia-0.3mm, flyingcarsfootprints:StitchingVia-0.3mm, F.Cu at (67.8, 61.1)
- added STITCH28: StitchingVia-0.3mm, flyingcarsfootprints:StitchingVia-0.3mm, F.Cu at (67.8, 59.0)
- added STITCH29: StitchingVia-0.3mm, flyingcarsfootprints:StitchingVia-0.3mm, F.Cu at (84.5, 36.1)
- added STITCH29: StitchingVia-0.3mm, flyingcarsfootprints:StitchingVia-0.3mm, F.Cu at (60.4, 62.8)
- added STITCH29: StitchingVia-0.3mm, flyingcarsfootprints:StitchingVia-0.3mm, F.Cu at (58.3, 20.9)
- added STITCH29: StitchingVia-0.3mm, flyingcarsfootprints:StitchingVia-0.3mm, F.Cu at (74.9, 21.7)
- added STITCH29: StitchingVia-0.3mm, flyingcarsfootprints:StitchingVia-0.3mm, F.Cu at (64.8, 59.0)
- added STITCH29: StitchingVia-0.3mm, flyingcarsfootprints:StitchingVia-0.3mm, F.Cu at (64.8, 61.1)
- added STITCH29: StitchingVia-0.3mm, flyingcarsfootprints:StitchingVia-0.3mm, F.Cu at (60.4, 52.6)
- added STITCH29: StitchingVia-0.3mm, flyingcarsfootprints:StitchingVia-0.3mm, F.Cu at (74.9, 32.1)
- added STITCH3: StitchingVia-0.3mm, flyingcarsfootprints:StitchingVia-0.3mm, F.Cu at (92.2, 28.6)
- added STITCH4: StitchingVia-0.3mm, flyingcarsfootprints:StitchingVia-0.3mm, F.Cu at (92.2, 31.2)
- added STITCH5: StitchingVia-0.3mm, flyingcarsfootprints:StitchingVia-0.3mm, F.Cu at (92.2, 33.7)
- added STITCH6: StitchingVia-0.3mm, flyingcarsfootprints:StitchingVia-0.3mm, F.Cu at (92.2, 36.2)
- added STITCH7: StitchingVia-0.3mm, flyingcarsfootprints:StitchingVia-0.3mm, F.Cu at (92.2, 59.8)
- added STITCH7: StitchingVia-0.3mm, flyingcarsfootprints:StitchingVia-0.3mm, F.Cu at (92.2, 38.8)
- added STITCH8: StitchingVia-0.3mm, flyingcarsfootprints:StitchingVia-0.3mm, F.Cu at (92.2, 62.3)
- added STITCH9: StitchingVia-0.3mm, flyingcarsfootprints:StitchingVia-0.3mm, F.Cu at (92.2, 64.8)
- moved C10 15.3 mm to (62.4, 45.0), turned to 180 degrees
- moved C3 13.2 mm to (66.4, 35.0), turned to 90 degrees
- moved C1 12.9 mm to (64.9, 47.8), turned to 90 degrees
- moved C2 12.8 mm to (62.4, 41.0)
- moved C6 10.7 mm to (73.5, 35.1), turned to -90 degrees
- moved C4 10.5 mm to (72.5, 35.1), turned to -90 degrees
- moved C7 8.75 mm to (73.0, 47.8), turned to 90 degrees
- moved C11 8.17 mm to (74.0, 47.8), turned to 90 degrees
- moved C5 5.66 mm to (75.8, 41.1), turned to 180 degrees
- moved U1 4.16 mm to (69.0, 41.5), turned to 180 degrees
- moved REF** 3.35 mm to (67.5, 31.1), turned to 90 degrees
- moved REF** 2.85 mm to (71.8, 31.4)
- moved REF** 1.45 mm to (70.4, 57.0)
- moved REF** 1.19 mm to (70.3, 21.7)
Routing:
- net ui_in[3]/mio[11]: track 36.5 -> 91.9 mm, vias 2 -> 4
- net ~{ctrl_sel_rst}/mio[36]: track 96.3 -> 42.8 mm, vias 6 -> 2
- net vccd: track 25.9 -> 76.3 mm, vias 2 -> 4
- net mio[37]: track 85.6 -> 36.9 mm, vias 4 -> 2
- net mio[35]: track 79.1 -> 31.9 mm, vias 4 -> 2
- net ui_in[4]/mio[12]: track 40.6 -> 81.4 mm, vias 2 -> 4
- net uo_out[5]/mio[21]: track 11.5 -> 51.3 mm, vias 2 -> 4
- net uo_out[2]/mio[18]: track 23.6 -> 60.8 mm
- net uo_out[4]/mio[20]: track 20.0 -> 55.9 mm
- net uo_out[7]/mio[23]: track 7.20 -> 42.5 mm, vias 0 -> 2
- net ctrl_sel_inc/mio[34]: track 69.8 -> 37.2 mm, vias 4 -> 2
- net uo_out[6]/mio[22]: track 15.8 -> 48.1 mm
- net uo_out[1]/mio[17]: track 19.0 -> 48.9 mm
- net uo_out[0]/mio[16]: track 28.0 -> 57.1 mm
- net GND: track 104.5 -> 75.6 mm, vias 87 -> 31
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Other:
- board text added: "AISLER"
- board text added: "Caravel QFN breakout"
- board text added: "v2.3"
- board text removed: "Caravel QFN bkout"
- board text removed: "aisler.net"
- board text removed: "v2.2"

Commit message: BOM adjustements, PCBA files
Parts:
- U1: footprint TinyTapeout:QFN-64-1EP_9x9mm_P0.5mm_EP7.65x7.65mm_REDUCEDPASTE -> Package_DFN_QFN:QFN-64-1EP_9x9mm_P0.5mm_EP7.65x7.65mm
Routing:
- net vddio: track 49.2 -> 49.7 mm
Other:
- board size 45 x 57.5 mm -> 45 x 52.5 mm
