File: breakout-qfn/caravel-breakout-qfn.kicad_sch (KiCad schematic)
At the start: 13 parts, among them CON1 REF-182665-01, CON2 REF-182665-01, CON3 73251-1352, U1 Caravel_QFN_TT4

Commit message: BOM adjustements, PCBA files
Parts:
- C1, C10, C11, C2, C3, C4, C5, C6, C7: MPN (none) -> EMK105B7104KV-F; MPN_ALT (none) -> CL05B104KA5NNNC; SMARTBOM (none) -> 0.1u 0402 10%
- CON1, CON2: MPN (none) -> REF-182665-01; MPN_ALT (none) -> FH-00339 (or Harwin M20-7812045)
- CON3: now not fitted
Changed lines of the file:
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@@
+      (effects (font (size 1.27 1.27)) hide)
+    )
+    (property "MPN" "EMK105B7104KV-F" (at 153.67 68.58 0)
+      (effects (font (size 1.27 1.27)) hide)
+    )
+    (property "MPN_ALT" "CL05B104KA5NNNC" (at 153.67 68.58 0)
+      (effects (font (size 1.27 1.27)) hide)
+    )
+    (property "SMARTBOM" "0.1u 0402 10%" (at 153.67 68.58 0)
       (effects (font (size 1.27 1.27)) hide)
     )
@@
       (effects (font (size 1.27 1.27)) hide)
     )
+    (property "MPN" "EMK105B7104KV-F" (at 135.89 100.33 0)
+      (effects (font (size 1.27 1.27)) hide)
+    )
+    (property "MPN_ALT" "CL05B104KA5NNNC" (at 135.89 100.33 0)
+      (effects (font (size 1.27 1.27)) hide)
+    )
+    (property "SMARTBOM" "0.1u 0402 10%" (at 135.89 100.33 0)
+      (effects (font (size 1.27 1.27)) hide)
+    )
     (pin "1")
     (pin "2")
@@
       (effects (font (size 1.27 1.27)) hide)
     )
+    (property "MPN" "EMK105B7104KV-F" (at 153.67 86.36 0)
+      (effects (font (size 1.27 1.27)) hide)
+    )
+    (property "MPN_ALT" "CL05B104KA5NNNC" (at 153.67 86.36 0)
+      (effects (font (size 1.27 1.27)) hide)
+    )
+    (property "SMARTBOM" "0.1u 0402 10%" (at 153.67 86.36 0)
+      (effects (font (size 1.27 1.27)) hide)
+    )
     (pin "1")
     (pin "2")
@@
       (effects (font (size 1.27 1.27)) hide)
     )
+    (property "MPN" "EMK105B7104KV-F" (at 118.11 33.02 0)
+      (effects (font (size 1.27 1.27)) hide)
+    )
+    (property "MPN_ALT" "CL05B104KA5NNNC" (at 118.11 33.02 0)
+      (effects (font (size 1.27 1.27)) hide)
+    )
+    (property "SMARTBOM" "0.1u 0402 10%" (at 118.11 33.02 0)
+      (effects (font (size 1.27 1.27)) hide)
+    )
     (pin "1")
     (pin "2")
@@
       (effects (font (size 1.27 1.27)) hide)
     )
+    (property "MPN" "EMK105B7104KV-F" (at 33.02 100.33 0)
+      (effects (font (size 1.27 1.27)) hide)
+    )
+    (property "MPN_ALT" "CL05B104KA5NNNC" (at 33.02 100.33 0)
+      (effects (font (size 1.27 1.27)) hide)
+    )
+    (property "SMARTBOM" "0.1u 0402 10%" (at 33.02 100.33 0)
+      (effects (font (size 1.27 1.27)) hide)
+    )
     (pin "1")
     (pin "2")
@@
       (effects (font (size 1.27 1.27)) hide)
     )
+    (property "MPN" "EMK105B7104KV-F" (at 91.44 138.43 0)
+      (effects (font (size 1.27 1.27)) hide)
+    )
+    (property "MPN_ALT" "CL05B104KA5NNNC" (at 91.44 138.43 0)
+      (effects (font (size 1.27 1.27)) hide)
+    )
+    (property "SMARTBOM" "0.1u 0402 10%" (at 91.44 138.43 0)
+      (effects (font (size 1.27 1.27)) hide)
+    )
     (pin "1")
     (pin "2")
@@
       (effects (font (size 1.27 1.27)) hide)
     )
+    (property "MPN" "EMK105B7104KV-F" (at 34.29 50.8 0)
+      (effects (font (size 1.27 1.27)) hide)
+    )
+    (property "MPN_ALT" "CL05B104KA5NNNC" (at 34.29 50.8 0)
+      (effects (font (size 1.27 1.27)) hide)
+    )
+    (property "SMARTBOM" "0.1u 0402 10%" (at 34.29 50.8 0)
+      (effects (font (size 1.27 1.27)) hide)
+    )
     (pin "1")
     (pin "2")
@@
       (effects (font (size 1.27 1.27)) hide)
     )
+    (property "MPN" "EMK105B7104KV-F" (at 62.23 31.75 0)
+      (effects (font (size 1.27 1.27)) hide)
+    )
+    (property "MPN_ALT" "CL05B104KA5NNNC" (at 62.23 31.75 0)
+      (effects (font (size 1.27 1.27)) hide)
+    )
+    (property "SMARTBOM" "0.1u 0402 10%" (at 62.23 31.75 0)
+      (effects (font (size 1.27 1.27)) hide)
+    )
     (pin "1")
     (pin "2")
@@
       (effects (font (size 1.27 1.27)) hide)
     )
+    (property "MPN" "EMK105B7104KV-F" (at 46.99 105.41 0)
+      (effects (font (size 1.27 1.27)) hide)
+    )
+    (property "MPN_ALT" "CL05B104KA5NNNC" (at 46.99 105.41 0)
+      (effects (font (size 1.27 1.27)) hide)
+    )
+    (property "SMARTBOM" "0.1u 0402 10%" (at 46.99 105.41 0)
+      (effects (font (size 1.27 1.27)) hide)
+    )
     (pin "1")
     (pin "2")
@@
     )
     (property "Datasheet" "~" (at 213.36 50.8 0)
+      (effects (font (size 1.27 1.27)) hide)
+    )
+    (property "MPN" "REF-182665-01" (at 213.36 50.8 0)
+      (effects (font (size 1.27 1.27)) hide)
+    )
+    (property "MPN_ALT" "FH-00339 (or Harwin M20-7812045)" (at 213.36 50.8 0)
       (effects (font (size 1.27 1.27)) hide)
     )
@@
       (effects (font (size 1.27 1.27)) hide)
     )
+    (property "MPN" "REF-182665-01" (at 213.36 124.46 0)
+      (effects (font (size 1.27 1.27)) hide)
+    )
+    (property "MPN_ALT" "FH-00339 (or Harwin M20-7812045)" (at 213.36 124.46 0)
+      (effects (font (size 1.27 1.27)) hide)
+    )
     (pin "1")
     (pin "10")
@@
   )
   (symbol (lib_id "ok-connectors:SMA_TH") (at 99.06 175.26 0) (unit 1)
-    (in_bom yes) (on_board yes) (dnp no)
+    (in_bom yes) (on_board yes) (dnp yes)
     (property "Reference" "CON3" (at 93.98 168.91 0)
       (effects (font (size 1.27 1.27)))
